File: rx-new.sch (KiCad schematic (older format))
At the start: 84 parts, among them Q1 BC848, Q2 BC858, U1 TPS79101DBVREP, U2 SN74CBT3253, U3 AD797, U4 AD797, U5 NC7SZ00M5X, U6 OPA1662, U7 74AUP1G74, U8 74AUP1G74

Commit message: Added BAT64-04 at RF input
Parts:
- removed D1, D2: BAT42, Diode_THT:D_DO-35_SOD27_P7.62mm_Horizontal, symbol Diode:BAT42
- added D1: BAT64-04, Package_TO_SOT_SMD:SOT-23, symbol custom_library:BAT64-04
Other:
- note removed: "Need to be BAT64-04"
Changed lines of the file:
@@
 Wire Wire Line
 	2600 1450 3500 1450
-Text Notes 1350 2150 0    50   ~ 0
-Need to be BAT64-04
-Wire Wire Line
-	1950 1450 2200 1450
-Connection ~ 1950 1450
-Connection ~ 1700 1450
-Wire Wire Line
-	1700 1450 1950 1450
-$Comp
-L power:GND #PWR09
-U 1 1 5F674BBB
-P 1950 1750
-F 0 "#PWR09" H 1950 1500 50  0001 C CNN
-F 1 "GND" H 1955 1577 50  0001 C CNN
-F 2 "" H 1950 1750 50  0001 C CNN
-F 3 "" H 1950 1750 50  0001 C CNN
-	1    1950 1750
-	1    0    0    -1
-$EndComp
-$Comp
-L power:GND #PWR05
-U 1 1 5F672E8C
-P 1700 1750
-F 0 "#PWR05" H 1700 1500 50  0001 C CNN
-F 1 "GND" H 1705 1577 50  0001 C CNN
-F 2 "" H 1700 1750 50  0001 C CNN
-F 3 "" H 1700 1750 50  0001 C CNN
-	1    1700 1750
-	1    0    0    -1
-$EndComp
-$Comp
-L Diode:BAT42 D2
-U 1 1 5F66A798
-P 1950 1600
-F 0 "D2" V 1996 1521 50  0000 R CNN
-F 1 "BAT42" V 1905 1521 50  0000 R CNN
-F 2 "Diode_THT:D_DO-35_SOD27_P7.62mm_Horizontal" H 1950 1425 50  0001 C CNN
-F 3 "http://www.vishay.com/docs/85660/bat42.pdf" H 1950 1600 50  0001 C CNN
-	1    1950 1600
-	0    -1   -1   0
-$EndComp
-$Comp
-L Diode:BAT42 D1
-U 1 1 5F6685CF
-P 1700 1600
-F 0 "D1" V 1654 1679 50  0000 L CNN
-F 1 "BAT42" V 1745 1679 50  0000 L CNN
-F 2 "Diode_THT:D_DO-35_SOD27_P7.62mm_Horizontal" H 1700 1425 50  0001 C CNN
-F 3 "http://www.vishay.com/docs/85660/bat42.pdf" H 1700 1600 50  0001 C CNN
-	1    1700 1600
-	0    -1   1    0
-$EndComp
 Text GLabel 1250 1450 0    50   Input ~ 0
 RF_IN
 Wire Wire Line
 	1350 1450 1250 1450
-Wire Wire Line
-	1550 1450 1700 1450
 $Comp
 L power:GND #PWR013
@@
 Text Label 4000 7050 3    50   ~ 0
 -Vf
+Wire Wire Line
+	1550 1450 1800 1450
+$Comp
+L custom_library:BAT64-04 D1
+U 1 1 5F61AD7E
+P 1800 1600
+F 0 "D1" H 1350 1500 50  0000 L CNN
+F 1 "BAT64-04" H 1200 1400 50  0000 L CNN
+F 2 "Package_TO_SOT_SMD:SOT-23" H 1875 1725 50  0001 L CNN
+F 3 "http://www.diodes.com/_files/datasheets/ds11005.pdf" V 1950 1480 50  0001 C CNN
+	1    1800 1600
+	1    0    0    -1
+$EndComp
+$Comp
+L power:GND #PWR05
+U 1 1 5F672E8C
+P 1650 1900
+F 0 "#PWR05" H 1650 1650 50  0001 C CNN
+F 1 "GND" H 1655 1727 50  0001 C CNN
+F 2 "" H 1650 1900 50  0001 C CNN
+F 3 "" H 1650 1900 50  0001 C CNN
+	1    1650 1900
+	1    0    0    -1
+$EndComp
+$Comp
+L power:GND #PWR09
+U 1 1 5F674BBB
+P 1950 1900
+F 0 "#PWR09" H 1950 1650 50  0001 C CNN
+F 1 "GND" H 1955 1727 50  0001 C CNN
+F 2 "" H 1950 1900 50  0001 C CNN
+F 3 "" H 1950 1900 50  0001 C CNN
+	1    1950 1900
+	1    0    0    -1
+$EndComp
+Wire Wire Line
+	1800 1500 1800 1450
+Connection ~ 1800 1450
+Wire Wire Line
+	1800 1450 2200 1450
 $EndSCHEMATC

Commit message: Added connectors and made DRC happy
Parts:
- added J1: RF_IN, Connector_Coaxial:SMA_Amphenol_901-144_Vertical, symbol Connector:Conn_Coaxial
- added J2: PWR_IN, symbol Connector:Conn_01x02_Male
- added J3: IQ_OUT, symbol Connector:AudioJack2_Ground
- added J4: 4LO_IN, Connector_Coaxial:SMA_Amphenol_901-144_Vertical, symbol Connector:Conn_Coaxial
Connections:
- net labels added: AUDIO_I, AUDIO_Q
- net labels removed: 4LO_IN, I, Q, RF_IN
- wire segments 245 -> 254
Other:
- note added: "Keep DRC happy"
Changed lines of the file:
@@
 	1    0    0    -1
 $EndComp
-Text GLabel 1350 5500 0    50   Input ~ 0
-Vbat
 Text Notes 3850 4350 0    50   ~ 0
 Power section
@@
 Wire Wire Line
 	2600 1450 3500 1450
-Text GLabel 1250 1450 0    50   Input ~ 0
-RF_IN
-Wire Wire Line
-	1350 1450 1250 1450
+Wire Wire Line
+	1350 1450 1200 1450
 $Comp
 L power:GND #PWR013
@@
 	1    0    0    -1
 $EndComp
-Text GLabel 1800 3700 1    50   Input ~ 0
-Vbat
 $Comp
 L Device:R_Small_US R1
@@
 	0    1    1    0
 $EndComp
-Text GLabel 7050 5500 0    50   Input ~ 0
-4LO_IN
 $Comp
 L Amplifier_Operational:OPA1602 U6
@@
 	0    -1   -1   0
 $EndComp
-Text GLabel 9050 1650 2    50   Output ~ 0
-I
 $Comp
 L Device:R_Small_US R21
@@
 	0    -1   -1   0
 $EndComp
-Text GLabel 9050 3350 2    50   Output ~ 0
-Q
 $Comp
 L Device:R_Small_US R22
@@
 Wire Wire Line
 	1800 1450 2200 1450
+$Comp
+L Connector:Conn_Coaxial J1
+U 1 1 5F6616CA
+P 1000 1450
+F 0 "J1" H 928 1688 50  0000 C CNN
+F 1 "RF_IN" H 928 1597 50  0000 C CNN
+F 2 "Connector_Coaxial:SMA_Amphenol_901-144_Vertical" H 1000 1450 50  0001 C CNN
+F 3 " ~" H 1000 1450 50  0001 C CNN
+	1    1000 1450
+	-1   0    0    -1
+$EndComp
+$Comp
+L power:GND #PWR041
+U 1 1 5F6844A3
+P 1000 1650
+F 0 "#PWR041" H 1000 1400 50  0001 C CNN
+F 1 "GND" H 1005 1477 50  0001 C CNN
+F 2 "" H 1000 1650 50  0001 C CNN
+F 3 "" H 1000 1650 50  0001 C CNN
+	1    1000 1650
+	1    0    0    -1
+$EndComp
+Wire Wire Line
+	1800 3700 1800 3550
+Text Label 1800 3550 0    50   ~ 0
+Vbat
+Text Label 1350 5500 2    50   ~ 0
+Vbat
+$Comp
+L Connector:Conn_01x02_Male J2
+U 1 1 5F6A93DD
+P 4700 5500
+F 0 "J2" H 4850 5750 50  0000 C CNN
+F 1 "PWR_IN" H 4850 5650 50  0000 C CNN
+F 2 "" H 4700 5500 50  0001 C CNN
+F 3 "~" H 4700 5500 50  0001 C CNN
+	1    4700 5500
+	1    0    0    -1
+$EndComp
+Wire Wire Line
+	4900 5500 5000 5500
+$Comp
+L power:GND #PWR043
+U 1 1 5F6BAE9C
+P 4900 5600
+F 0 "#PWR043" H 4900 5350 50  0001 C CNN
+F 1 "GND" H 4905 5427 50  0001 C CNN
+F 2 "" H 4900 5600 50  0001 C CNN
+F 3 "" H 4900 5600 50  0001 C CNN
+	1    4900 5600
+	0    -1   -1   0
+$EndComp
+Text Label 5000 5500 0    50   ~ 0
+Vbat
+$Comp
+L Connector:AudioJack2_Ground J3
+U 1 1 5F6BD3CF
+P 4800 6100
+F 0 "J3" H 4832 6425 50  0000 C CNN
+F 1 "IQ_OUT" H 4832 6334 50  0000 C CNN
+F 2 "" H 4800 6100 50  0001 C CNN
+F 3 "~" H 4800 6100 50  0001 C CNN
+	1    4800 6100
+	1    0    0    -1
+$EndComp
+Wire Wire Line
+	5000 6000 5050 6000
+Wire Wire Line
+	5000 6100 5050 6100
+$Comp
+L power:GND #PWR042
+U 1 1 5F6E0D11
+P 4800 6300
+F 0 "#PWR042" H 4800 6050 50  0001 C CNN
+F 1 "GND" H 4805 6127 50  0001 C CNN
+F 2 "" H 4800 6300 50  0001 C CNN
+F 3 "" H 4800 6300 50  0001 C CNN
+	1    4800 6300
+	1    0    0    -1
+$EndComp
+Text Label 5050 6000 0    50   ~ 0
+AUDIO_I
+Text Label 5050 6100 0    50   ~ 0
+AUDIO_Q
+$Comp
+L Connector:Conn_Coaxial J4
+U 1 1 5F6F3F62
+P 6850 5500
+F 0 "J4" H 6778 5738 50  0000 C CNN
+F 1 "4LO_IN" H 6778 5647 50  0000 C CNN
+F 2 "Connector_Coaxial:SMA_Amphenol_901-144_Vertical" H 6850 5500 50  0001 C CNN
+F 3 " ~" H 6850 5500 50  0001 C CNN
+	1    6850 5500
+	-1   0    0    -1
+$EndComp
+$Comp
+L power:GND #PWR044
+U 1 1 5F7056D4
+P 6850 5700
+F 0 "#PWR044" H 6850 5450 50  0001 C CNN
+F 1 "GND" H 6855 5527 50  0001 C CNN
+F 2 "" H 6850 5700 50  0001 C CNN
+F 3 "" H 6850 5700 50  0001 C CNN
+	1    6850 5700
+	1    0    0    -1
+$EndComp
+Wire Wire Line
+	9050 1650 9150 1650
+Wire Wire Line
+	9050 3350 9150 3350
+Text Label 9150 1650 0    50   ~ 0
+AUDIO_I
+Text Label 9150 3350 0    50   ~ 0
+AUDIO_Q
+$Comp
+L power:PWR_FLAG #FLG0101
+U 1 1 5F72BF33
+P 5200 6950
+F 0 "#FLG0101" H 5200 7025 50  0001 C CNN
+F 1 "PWR_FLAG" H 5200 7123 50  0001 C CNN
+F 2 "" H 5200 6950 50  0001 C CNN
+F 3 "~" H 5200 6950 50  0001 C CNN
+	1    5200 6950
+	1    0    0    -1
+$EndComp
+$Comp
+L power:GND #PWR0101
+U 1 1 5F72D5F9
+P 5200 6950
+F 0 "#PWR0101" H 5200 6700 50  0001 C CNN
+F 1 "GND" H 5205 6777 50  0001 C CNN
+F 2 "" H 5200 6950 50  0001 C CNN
+F 3 "" H 5200 6950 50  0001 C CNN
+	1    5200 6950
+	1    0    0    -1
+$EndComp
+$Comp
+L power:PWR_FLAG #FLG0102
+U 1 1 5F72DB65
+P 5350 6950
+F 0 "#FLG0102" H 5350 7025 50  0001 C CNN
+F 1 "PWR_FLAG" H 5350 7123 50  0001 C CNN
+F 2 "" H 5350 6950 50  0001 C CNN
+F 3 "~" H 5350 6950 50  0001 C CNN
+	1    5350 6950
+	1    0    0    -1
+$EndComp
+Wire Wire Line
+	5350 6950 5350 7050
+Text Label 5350 7050 0    50   ~ 0
+Vbat
+Text Notes 5200 6800 0    50   ~ 0
+Keep DRC happy
+$Comp
+L power:PWR_FLAG #FLG0103
+U 1 1 5F763F49
+P 5600 6950
+F 0 "#FLG0103" H 5600 7025 50  0001 C CNN
+F 1 "PWR_FLAG" H 5600 7123 50  0001 C CNN
+F 2 "" H 5600 6950 50  0001 C CNN
+F 3 "~" H 5600 6950 50  0001 C CNN
+	1    5600 6950
+	1    0    0    -1
+$EndComp
+Wire Wire Line
+	5600 6950 5600 7050
+Text Label 5600 7050 0    50   ~ 0
+-Vf
+$Comp
+L power:PWR_FLAG #FLG0104
+U 1 1 5F776F7E
+P 5800 6950
+F 0 "#FLG0104" H 5800 7025 50  0001 C CNN
+F 1 "PWR_FLAG" H 5800 7123 50  0001 C CNN
+F 2 "" H 5800 6950 50  0001 C CNN
+F 3 "~" H 5800 6950 50  0001 C CNN
+	1    5800 6950
+	1    0    0    -1
+$EndComp
+Wire Wire Line
+	5800 6950 5800 7050
+Text Label 5800 7050 0    50   ~ 0
++Vd
 $EndSCHEMATC

Commit message: enable_LCL_Less_elco
Parts:
- removed C33, C41, C44, C45: 47u, symbol Device:CP_Small
- added C? (x2): 1n, symbol Device:C_Small
- added C?: 0.1u, symbol Device:C_Small
- added C?: 47u, symbol Device:CP_Small
- added L?: L, symbol Device:L
- added Q?: BC848, Package_TO_SOT_SMD:SOT-23, symbol Transistor_BJT:BC848
- added Q?: BC858, Package_TO_SOT_SMD:SOT-23, symbol Transistor_BJT:BC858
- added R? (x2): 10k, symbol Device:R_Small_US
- added R?: 100k, symbol Device:R_Small_US
- added R?: 47k, symbol Device:R_Small_US
Connections:
- net labels added: En, Eo
Other:
- moved on the sheet: J3

Commit message: Modified CLC to CLCLC, updated libraries, added En pin to power input connector
Parts:
- removed J2: PWR_IN, symbol Connector:Conn_01x02_Male
- added C48: 47u, symbol Device:CP_Small
- added J2: PWR_IN, symbol Connector:Conn_01x03_Male
- added L1: 10uH, Inductor_SMD:L_0805_2012Metric_Pad1.15x1.40mm_HandSolder, symbol Device:L
- C1, C10, C11, C13, C14, C15, C16, C17, C2, C21, C22, C25, C26, C27, C28, C29, C3, C31, C32, C34, C35, C36, C37, C39, C4, C40, C42, C43, C46, C47, C5, C7, C8: footprint (none) -> Capacitor_SMD:C_0805_2012Metric_Pad1.15x1.40mm_HandSolder
- C33, C41, C44: renamed from C?; footprint (none) -> Capacitor_SMD:C_0805_2012Metric_Pad1.15x1.40mm_HandSolder
- L2: renamed from L?; value L -> 10uH; footprint (none) -> Inductor_SMD:L_0805_2012Metric_Pad1.15x1.40mm_HandSolder
- R1, R10, R11, R13, R14, R15, R16, R17, R18, R19, R2, R21, R22, R23, R24, R3, R4, R5, R6, R7, R8, R9: footprint (none) -> Resistor_SMD:R_0805_2012Metric_Pad1.15x1.40mm_HandSolder
- R25, R26, R27, R28: renamed from R?; footprint (none) -> Resistor_SMD:R_0805_2012Metric_Pad1.15x1.40mm_HandSolder
- gave numbers to parts that had none: 3
Connections:
- wire segments 254 -> 269
Other:
- moved on the sheet: L2, Q3, Q4, R25, R26, R27

Commit message: C48
Parts:
- removed C48: 47u, symbol Device:CP_Small
- added C48: 0.1u, Capacitor_SMD:C_0805_2012Metric_Pad1.15x1.40mm_HandSolder, symbol Device:C_Small
Connections:
- net GND: now also C48.1
- net at L1.2, L2.1: now also C48.2
Changed lines of the file:
@@
 EESchema Schematic File Version 4
-EELAYER 30 0
+LIBS:rx-new-cache
+EELAYER 29 0
 EELAYER END
 $Descr A4 11693 8268
@@
 	0    -1   -1   0
 $EndComp
-$Comp
-L Device:CP_Small C48
-U 1 1 5F7D5276
-P 5500 5700
-F 0 "C48" V 5500 5350 50  0000 L CNN
-F 1 "47u" V 5500 5150 50  0000 L CNN
-F 2 "" H 5500 5700 50  0001 C CNN
-F 3 "~" H 5500 5700 50  0001 C CNN
-	1    5500 5700
-	1    0    0    -1
-$EndComp
 Wire Wire Line
 	5500 5600 5500 5500
-$Comp
-L power:GND #PWR0111
-U 1 1 5F7D527D
-P 5500 5800
-F 0 "#PWR0111" H 5500 5550 50  0001 C CNN
-F 1 "GND" H 5505 5627 50  0001 C CNN
-F 2 "" H 5500 5800 50  0001 C CNN
-F 3 "" H 5500 5800 50  0001 C CNN
-	1    5500 5800
-	1    0    0    -1
-$EndComp
 Wire Wire Line
 	5450 5500 5500 5500
@@
 Wire Wire Line
 	3250 4100 3250 4150
+$Comp
+L Device:C_Small C48
+U 1 1 5FA5A39D
+P 5500 5700
+F 0 "C48" V 5500 6000 50  0000 C CNN
+F 1 "0.1u" V 5500 6200 50  0000 C CNN
+F 2 "Capacitor_SMD:C_0805_2012Metric_Pad1.15x1.40mm_HandSolder" H 5500 5700 50  0001 C CNN
+F 3 "~" H 5500 5700 50  0001 C CNN
+	1    5500 5700
+	-1   0    0    1
+$EndComp
+$Comp
+L power:GND #PWR?
+U 1 1 5FA5A3A3
+P 5500 5800
+F 0 "#PWR?" H 5500 5550 50  0001 C CNN
+F 1 "GND" H 5505 5627 50  0001 C CNN
+F 2 "" H 5500 5800 50  0001 C CNN
+F 3 "" H 5500 5800 50  0001 C CNN
+	1    5500 5800
+	1    0    0    -1
+$EndComp
 $EndSCHEMATC

Commit message: Added 1210 CP footprint and created custom symbol for audio jack
Parts:
- removed J3: IQ_OUT, symbol Connector:AudioJack2_Ground
- added J3: IQ_OUT, Connector_Audio:Jack_3.5mm_CUI_SJ1-3533NG_Horizontal, symbol custom_library:SJ1-3533NG
- C12: footprint (none) -> custom_library:CP_1210_3225Metric_Pad1.42x2.65mm_HandSolder; Mfr no. (none) -> F931C476MBAAJ6
- C18, C20, C30, C38, C45, C9: footprint (none) -> custom_library:CP_1210_3225Metric_Pad1.42x2.65mm_HandSolder
- C19, C6: footprint (none) -> custom_library:CP_1210_3225Metric_Pad1.42x2.65mm_HandSolder; Mfr no (none) -> F931C476MBAAJ6
- C23, C24: footprint (none) -> Capacitor_SMD:C_0805_2012Metric_Pad1.15x1.40mm_HandSolder
- J2: footprint (none) -> Connector_PinHeader_2.54mm:PinHeader_1x03_P2.54mm_Vertical
- R12, R20: footprint (none) -> Resistor_SMD:R_0805_2012Metric_Pad1.15x1.40mm_HandSolder
- U1: footprint Texas_Instruments-TPS79101DBVREP-* -> custom_library:Texas_Instruments-TPS79101DBVREP-Level_A; MPN (none) -> TPS79101DBVREP
Connections:
- net AUDIO_I: now also J3.R
- net AUDIO_Q: now also J3.T
- net GND: now also J3.S
Changed lines of the file:
@@
 EESchema Schematic File Version 4
-LIBS:rx-new-cache
-EELAYER 29 0
+EELAYER 30 0
 EELAYER END
 $Descr A4 11693 8268
@@
 F 0 "C20" V 4150 550 50  0000 L CNN
 F 1 "47u" V 4150 350 50  0000 L CNN
-F 2 "" H 4150 1000 50  0001 C CNN
+F 2 "custom_library:CP_1210_3225Metric_Pad1.42x2.65mm_HandSolder" H 4150 1000 50  0001 C CNN
 F 3 "~" H 4150 1000 50  0001 C CNN
 	1    4150 1000
@@
 F 0 "C19" V 3750 6500 50  0000 L CNN
 F 1 "47u" V 3750 6300 50  0000 L CNN
-F 2 "" H 3750 6950 50  0001 C CNN
+F 2 "custom_library:CP_1210_3225Metric_Pad1.42x2.65mm_HandSolder" H 3750 6950 50  0001 C CNN
 F 3 "~" H 3750 6950 50  0001 C CNN
+F 4 "F931C476MBAAJ6" V 3750 6950 50  0001 C CNN "Mfr no"
 	1    3750 6950
 	1    0    0    -1
@@
 F 0 "C18" V 3650 5350 50  0000 L CNN
 F 1 "47u" V 3650 5150 50  0000 L CNN
-F 2 "" H 3650 5700 50  0001 C CNN
+F 2 "custom_library:CP_1210_3225Metric_Pad1.42x2.65mm_HandSolder" H 3650 5700 50  0001 C CNN
 F 3 "~" H 3650 5700 50  0001 C CNN
 	1    3650 5700
@@
 F 0 "C12" V 2600 6500 50  0000 L CNN
 F 1 "47u" V 2600 6300 50  0000 L CNN
-F 2 "" H 2600 6850 50  0001 C CNN
+F 2 "custom_library:CP_1210_3225Metric_Pad1.42x2.65mm_HandSolder" H 2600 6850 50  0001 C CNN
 F 3 "~" H 2600 6850 50  0001 C CNN
+F 4 "F931C476MBAAJ6" V 2600 6850 50  0001 C CNN "Mfr no."
 	1    2600 6850
 	1    0    0    -1
@@
 F 0 "U1" H 2350 5765 50  0000 C CNN
 F 1 "TPS79101DBVREP" H 2350 5674 50  0000 C CNN
-F 2 "Texas_Instruments-TPS79101DBVREP-*" H 1850 5900 50  0001 L CNN
+F 2 "custom_library:Texas_Instruments-TPS79101DBVREP-Level_A" H 1850 5900 50  0001 L CNN
 F 3 "http://www.ti.com/general/docs/lit/getliterature.tsp?genericPartNumber=TPS79101-EP&fileType=pdf" H 1850 6000 50  0001 L CNN
 F 4 "2" H 1850 6100 50  0001 L CNN "Accuracy"
@@
 F 29 "E89202BC-B87B-4135-AE28-EC4511A6FCC2" H 1850 8600 50  0001 L CNN "vault revision"
 F 30 "yes" H 1850 8700 50  0001 L CNN "imported"
+F 31 "TPS79101DBVREP" H 1850 5500 50  0001 C CNN "MPN"
 	1    1850 5500
 	1    0    0    -1
@@
 F 0 "C24" V 4150 3150 50  0000 C CNN
 F 1 "0.1u" V 4150 3300 50  0000 C CNN
-F 2 "" H 4150 2850 50  0001 C CNN
+F 2 "Capacitor_SMD:C_0805_2012Metric_Pad1.15x1.40mm_HandSolder" H 4150 2850 50  0001 C CNN
 F 3 "~" H 4150 2850 50  0001 C CNN
 	1    4150 2850
@@
 F 0 "C23" V 4150 3000 50  0000 C CNN
 F 1 "1n" V 4150 3150 50  0000 C CNN
-F 2 "" H 4150 2700 50  0001 C CNN
+F 2 "Capacitor_SMD:C_0805_2012Metric_Pad1.15x1.40mm_HandSolder" H 4150 2700 50  0001 C CNN
 F 3 "~" H 4150 2700 50  0001 C CNN
 	1    4150 2700
@@
 F 0 "C9" V 2100 4400 50  0000 L CNN
 F 1 "47u" V 2100 4250 50  0000 L CNN
-F 2 "" H 2100 4700 50  0001 C CNN
+F 2 "custom_library:CP_1210_3225Metric_Pad1.42x2.65mm_HandSolder" H 2100 4700 50  0001 C CNN
 F 3 "~" H 2100 4700 50  0001 C CNN
 	1    2100 4700
@@
 F 0 "C6" V 1750 5350 50  0000 L CNN
 F 1 "47u" V 1750 5150 50  0000 L CNN
-F 2 "" H 1750 5700 50  0001 C CNN
+F 2 "custom_library:CP_1210_3225Metric_Pad1.42x2.65mm_HandSolder" H 1750 5700 50  0001 C CNN
 F 3 "~" H 1750 5700 50  0001 C CNN
+F 4 "F931C476MBAAJ6" V 1750 5700 50  0001 C CNN "Mfr no"
 	1    1750 5700
 	1    0    0    -1
@@
 F 0 "R12" V 7300 2050 50  0000 C CNN
 F 1 "1E" V 7300 2350 50  0000 C CNN
-F 2 "" H 7350 2200 50  0001 C CNN
+F 2 "Resistor_SMD:R_0805_2012Metric_Pad1.15x1.40mm_HandSolder" H 7350 2200 50  0001 C CNN
 F 3 "~" H 7350 2200 50  0001 C CNN
 	1    7350 2200
@@
 F 0 "R20" V 7795 6050 50  0000 C CNN
 F 1 "22k" V 7886 6050 50  0000 C CNN
-F 2 "" H 8000 6050 50  0001 C CNN
+F 2 "Resistor_SMD:R_0805_2012Metric_Pad1.15x1.40mm_HandSolder" H 8000 6050 50  0001 C CNN
 F 3 "~" H 8000 6050 50  0001 C CNN
 	1    8000 6050
@@
 F 0 "C38" V 7850 4950 50  0000 L CNN
 F 1 "47u" V 7850 5550 50  0000 L CNN
-F 2 "" H 7850 5300 50  0001 C CNN
+F 2 "custom_library:CP_1210_3225Metric_Pad1.42x2.65mm_HandSolder" H 7850 5300 50  0001 C CNN
 F 3 "~" H 7850 5300 50  0001 C CNN
 	1    7850 5300
@@
 F 0 "C30" V 7350 600 50  0000 L CNN
 F 1 "47u" V 7350 400 50  0000 L CNN
-F 2 "" H 7350 1050 50  0001 C CNN
+F 2 "custom_library:CP_1210_3225Metric_Pad1.42x2.65mm_HandSolder" H 7350 1050 50  0001 C CNN
 F 3 "~" H 7350 1050 50  0001 C CNN
 	1    7350 1050
@@
 Text Label 5850 5500 0    50   ~ 0
 Vbat
-$Comp
-L Connector:AudioJack2_Ground J3
-U 1 1 5F6BD3CF
-P 9000 2500
-F 0 "J3" H 9032 2825 50  0000 C CNN
-F 1 "IQ_OUT" H 9032 2734 50  0000 C CNN
-F 2 "" H 9000 2500 50  0001 C CNN
-F 3 "~" H 9000 2500 50  0001 C CNN
-	1    9000 2500
-	1    0    0    -1
-$EndComp
 Wire Wire Line
 	9200 2400 9250 2400
@@
 F 0 "C45" V 5100 5350 50  0000 L CNN
 F 1 "47u" V 5100 5150 50  0000 L CNN
-F 2 "" H 5100 5700 50  0001 C CNN
+F 2 "custom_library:CP_1210_3225Metric_Pad1.42x2.65mm_HandSolder" H 5100 5700 50  0001 C CNN
 F 3 "~" H 5100 5700 50  0001 C CNN
 	1    5100 5700
@@
 F 0 "J2" H 4500 5950 50  0000 C CNN
 F 1 "PWR_IN" H 4500 5850 50  0000 C CNN
-F 2 "" H 4400 5600 50  0001 C CNN
+F 2 "Connector_PinHeader_2.54mm:PinHeader_1x03_P2.54mm_Vertical" H 4400 5600 50  0001 C CNN
 F 3 "~" H 4400 5600 50  0001 C CNN
 	1    4400 5600
@@
 $EndComp
 $Comp
-L power:GND #PWR?
+L power:GND #PWR0111
 U 1 1 5FA5A3A3
 P 5500 5800
-F 0 "#PWR?" H 5500 5550 50  0001 C CNN
+F 0 "#PWR0111" H 5500 5550 50  0001 C CNN
 F 1 "GND" H 5505 5627 50  0001 C CNN
 F 2 "" H 5500 5800 50  0001 C CNN
@@
 	1    0    0    -1
 $EndComp
+$Comp
+L custom_library:SJ1-3533NG J3
+U 1 1 5F6E4CFB
+P 9000 2500
+F 0 "J3" H 9032 2825 50  0000 C CNN
+F 1 "IQ_OUT" H 9032 2734 50  0000 C CNN
+F 2 "Connector_Audio:Jack_3.5mm_CUI_SJ1-3533NG_Horizontal" H 9000 2500 50  0001 C CNN
+F 3 "https://ro.mouser.com/datasheet/2/670/sj1_353xng-1778850.pdf" H 9000 2500 50  0001 C CNN
+F 4 "SJ1-3533NG" H 9000 2500 50  0001 C CNN "MPN"
+	1    9000 2500
+	1    0    0    -1
+$EndComp
