File: rx-new.sch (KiCad schematic (older format))
At the start: 96 parts, among them J1 RF_IN, J2 PWR_IN, J3 IQ_OUT, J4 4LO_IN, Q1 BC848, Q2 BC858, Q3 BC848, Q4 BC858, U1 TPS79101DBVREP, U2 SN74CBT3253, U3 AD797, U4 AD797, U5 NC7SZ00M5X, U6 OPA1662, U7 74AUP1G74, U8 74AUP1G74

Commit message: finished_layout
Parts:
- C42: value 0.1u -> 1n
Connections:
- net +Vd: no longer C42.2
- net -Vf: now also C42.2; no longer C42.1
- net GND: now also C42.1
- net at U2.7 (1A): now also TR1.6; no longer TR1.4
- net at U2.9 (2A): now also TR1.4; no longer TR1.6
Other:
- moved on the sheet: C2, C33, C42, D1, J1
Changed lines of the file:
@@
 EESchema Schematic File Version 4
-EELAYER 30 0
+LIBS:rx-new-cache
+EELAYER 29 0
 EELAYER END
 $Descr A4 11693 8268
@@
 Wire Wire Line
 	2450 6650 2300 6650
-Wire Wire Line
-	2600 6650 2700 6650
 Connection ~ 2600 6650
 $Comp
@@
 	2600 1450 3500 1450
 Wire Wire Line
-	1350 1450 1200 1450
+	1350 1850 1200 1850
 $Comp
 L power:GND #PWR013
 U 1 1 5F5A3FE3
-P 2200 1850
-F 0 "#PWR013" H 2200 1600 50  0001 C CNN
-F 1 "GND" H 2205 1677 50  0001 C CNN
-F 2 "" H 2200 1850 50  0001 C CNN
-F 3 "" H 2200 1850 50  0001 C CNN
-	1    2200 1850
+P 2200 1450
+F 0 "#PWR013" H 2200 1200 50  0001 C CNN
+F 1 "GND" H 2205 1277 50  0001 C CNN
+F 2 "" H 2200 1450 50  0001 C CNN
+F 3 "" H 2200 1450 50  0001 C CNN
+	1    2200 1450
 	0    1    1    0
 $EndComp
@@
 L Device:C_Small C2
 U 1 1 5F58E35D
-P 1450 1450
-F 0 "C2" V 1221 1450 50  0000 C CNN
-F 1 "0.1u" V 1312 1450 50  0000 C CNN
-F 2 "Capacitor_SMD:C_0805_2012Metric_Pad1.15x1.40mm_HandSolder" H 1450 1450 50  0001 C CNN
-F 3 "~" H 1450 1450 50  0001 C CNN
-	1    1450 1450
+P 1450 1850
+F 0 "C2" V 1221 1850 50  0000 C CNN
+F 1 "0.1u" V 1312 1850 50  0000 C CNN
+F 2 "Capacitor_SMD:C_0805_2012Metric_Pad1.15x1.40mm_HandSolder" H 1450 1850 50  0001 C CNN
+F 3 "~" H 1450 1850 50  0001 C CNN
+	1    1450 1850
 	0    1    1    0
 $EndComp
@@
 F 3 "https://www.minicircuits.com/pdfs/ADT4-6WT+.pdf" H 2400 1650 50  0001 C CNN
 	1    2400 1650
-	1    0    0    -1
+	1    0    0    1
 $EndComp
 Wire Wire Line
@@
 L Device:C_Small C42
 U 1 1 5F7B403A
-P 9700 4800
-F 0 "C42" V 9700 4550 50  0000 C CNN
-F 1 "0.1u" V 9700 4300 50  0000 C CNN
-F 2 "Capacitor_SMD:C_0805_2012Metric_Pad1.15x1.40mm_HandSolder" H 9700 4800 50  0001 C CNN
-F 3 "~" H 9700 4800 50  0001 C CNN
-	1    9700 4800
-	0    -1   -1   0
+P 3000 6850
+F 0 "C42" V 3000 6600 50  0000 C CNN
+F 1 "1n" V 3000 6350 50  0000 C CNN
+F 2 "Capacitor_SMD:C_0805_2012Metric_Pad1.15x1.40mm_HandSolder" H 3000 6850 50  0001 C CNN
+F 3 "~" H 3000 6850 50  0001 C CNN
+	1    3000 6850
+	-1   0    0    1
 $EndComp
 Wire Wire Line
@@
 -Vf
 Wire Wire Line
-	1550 1450 1800 1450
+	1550 1850 1800 1850
 $Comp
 L custom_library:BAT64-04 D1
 U 1 1 5F61AD7E
-P 1800 1600
-F 0 "D1" H 1600 1150 50  0000 L CNN
-F 1 "BAT64-04" H 1750 1150 50  0000 L CNN
-F 2 "Package_TO_SOT_SMD:SOT-23" H 1875 1725 50  0001 L CNN
-F 3 "http://www.diodes.com/_files/datasheets/ds11005.pdf" V 1950 1480 50  0001 C CNN
-	1    1800 1600
+P 1800 2000
+F 0 "D1" H 1600 1550 50  0000 L CNN
+F 1 "BAT64-04" H 1750 1550 50  0000 L CNN
+F 2 "Package_TO_SOT_SMD:SOT-23" H 1875 2125 50  0001 L CNN
+F 3 "http://www.diodes.com/_files/datasheets/ds11005.pdf" V 1950 1880 50  0001 C CNN
+	1    1800 2000
 	1    0    0    -1
 $EndComp
@@
 L power:GND #PWR05
 U 1 1 5F672E8C
-P 1650 1900
-F 0 "#PWR05" H 1650 1650 50  0001 C CNN
-F 1 "GND" H 1655 1727 50  0001 C CNN
-F 2 "" H 1650 1900 50  0001 C CNN
-F 3 "" H 1650 1900 50  0001 C CNN
-	1    1650 1900
+P 1650 2300
+F 0 "#PWR05" H 1650 2050 50  0001 C CNN
+F 1 "GND" H 1655 2127 50  0001 C CNN
+F 2 "" H 1650 2300 50  0001 C CNN
+F 3 "" H 1650 2300 50  0001 C CNN
+	1    1650 2300
 	1    0    0    -1
 $EndComp
@@
 L power:GND #PWR09
 U 1 1 5F674BBB
-P 1950 1900
-F 0 "#PWR09" H 1950 1650 50  0001 C CNN
-F 1 "GND" H 1955 1727 50  0001 C CNN
-F 2 "" H 1950 1900 50  0001 C CNN
-F 3 "" H 1950 1900 50  0001 C CNN
-	1    1950 1900
-	1    0    0    -1
-$EndComp
-Wire Wire Line
-	1800 1500 1800 1450
-Connection ~ 1800 1450
-Wire Wire Line
-	1800 1450 2200 1450
+P 1950 2300
+F 0 "#PWR09" H 1950 2050 50  0001 C CNN
+F 1 "GND" H 1955 2127 50  0001 C CNN
+F 2 "" H 1950 2300 50  0001 C CNN
+F 3 "" H 1950 2300 50  0001 C CNN
+	1    1950 2300
+	1    0    0    -1
+$EndComp
+Wire Wire Line
+	1800 1900 1800 1850
+Connection ~ 1800 1850
+Wire Wire Line
+	1800 1850 2200 1850
 $Comp
 L Connector:Conn_Coaxial J1
 U 1 1 5F6616CA
-P 1000 1450
-F 0 "J1" H 928 1688 50  0000 C CNN
-F 1 "RF_IN" H 928 1597 50  0000 C CNN
-F 2 "Connector_Coaxial:SMA_Amphenol_901-144_Vertical" H 1000 1450 50  0001 C CNN
-F 3 " ~" H 1000 1450 50  0001 C CNN
-	1    1000 1450
+P 1000 1850
+F 0 "J1" H 928 2088 50  0000 C CNN
+F 1 "RF_IN" H 928 1997 50  0000 C CNN
+F 2 "Connector_Coaxial:SMA_Amphenol_901-144_Vertical" H 1000 1850 50  0001 C CNN
+F 3 " ~" H 1000 1850 50  0001 C CNN
+	1    1000 1850
 	-1   0    0    -1
 $EndComp
@@
 L power:GND #PWR041
 U 1 1 5F6844A3
-P 1000 1650
-F 0 "#PWR041" H 1000 1400 50  0001 C CNN
-F 1 "GND" H 1005 1477 50  0001 C CNN
-F 2 "" H 1000 1650 50  0001 C CNN
-F 3 "" H 1000 1650 50  0001 C CNN
-	1    1000 1650
+P 1000 2050
+F 0 "#PWR041" H 1000 1800 50  0001 C CNN
+F 1 "GND" H 1005 1877 50  0001 C CNN
+F 2 "" H 1000 2050 50  0001 C CNN
+F 3 "" H 1000 2050 50  0001 C CNN
+	1    1000 2050
 	1    0    0    -1
 $EndComp
@@
 L Device:C_Small C33
 U 1 1 5F90581F
-P 1450 1600
-F 0 "C33" V 1300 1600 50  0000 C CNN
-F 1 "1n" V 1200 1600 50  0000 C CNN
-F 2 "Capacitor_SMD:C_0805_2012Metric_Pad1.15x1.40mm_HandSolder" H 1450 1600 50  0001 C CNN
-F 3 "~" H 1450 1600 50  0001 C CNN
-	1    1450 1600
-	0    -1   -1   0
-$EndComp
-Wire Wire Line
-	1550 1600 1550 1450
-Connection ~ 1550 1450
-Wire Wire Line
-	1350 1600 1350 1450
-Connection ~ 1350 1450
+P 1450 2000
+F 0 "C33" V 1300 2000 50  0000 C CNN
+F 1 "1n" V 1200 2000 50  0000 C CNN
+F 2 "Capacitor_SMD:C_0805_2012Metric_Pad1.15x1.40mm_HandSolder" H 1450 2000 50  0001 C CNN
+F 3 "~" H 1450 2000 50  0001 C CNN
+	1    1450 2000
+	0    -1   -1   0
+$EndComp
+Wire Wire Line
+	1550 2000 1550 1850
+Connection ~ 1550 1850
+Wire Wire Line
+	1350 2000 1350 1850
+Connection ~ 1350 1850
 $Comp
 L power:GND #PWR0102
@@
 	1    0    0    -1
 $EndComp
+$Comp
+L power:GND #PWR?
+U 1 1 5F9C6168
+P 3000 6950
+F 0 "#PWR?" H 3000 6700 50  0001 C CNN
+F 1 "GND" H 3005 6777 50  0001 C CNN
+F 2 "" H 3000 6950 50  0001 C CNN
+F 3 "" H 3000 6950 50  0001 C CNN
+	1    3000 6950
+	1    0    0    -1
+$EndComp
+Wire Wire Line
+	3000 6750 3000 6650
+Wire Wire Line
+	2600 6650 3000 6650
 $EndSCHEMATC

Commit message: Fixed audio jack pin assignment
Connections:
- net AUDIO_I: now also J3.T; no longer J3.R
- net AUDIO_Q: now also J3.R; no longer J3.T
Changed lines of the file:
@@
 EESchema Schematic File Version 4
-LIBS:rx-new-cache
-EELAYER 29 0
+EELAYER 30 0
 EELAYER END
 $Descr A4 11693 8268
@@
 $EndComp
 Text Label 9250 2400 0    50   ~ 0
+AUDIO_Q
+Text Label 9250 2500 0    50   ~ 0
 AUDIO_I
-Text Label 9250 2500 0    50   ~ 0
-AUDIO_Q
 $Comp
 L Connector:Conn_Coaxial J4
@@
 $EndComp
 $Comp
-L power:GND #PWR?
+L power:GND #PWR0112
 U 1 1 5F9C6168
 P 3000 6950
-F 0 "#PWR?" H 3000 6700 50  0001 C CNN
+F 0 "#PWR0112" H 3000 6700 50  0001 C CNN
 F 1 "GND" H 3005 6777 50  0001 C CNN
 F 2 "" H 3000 6950 50  0001 C CNN
